Commit message: Robotiq installation

File: urdf/camera.xacro (robot description, xacro)
@@ -18,5 +18,5 @@
         <collision>
             <geometry>
-                <mesh filename="package://ur5_sim/meshes/sensors/camera/kinetic.dae"/>
+                <mesh filename="package://ur5_sim/meshes/sensors/camera/kinetic.stl"/>
             </geometry>
         </collision>
@@ -57,3 +57,11 @@
         </sensor>
     </gazebo>
+    <gazebo reference="camera_link">
+        <visual>
+            <geometry>
+                <mesh filename="package://ur5_sim/meshes/sensors/camera/kinetic.stl"/>
+            </geometry>
+            <material>Gazebo/Red</material>
+        </visual>
+    </gazebo>
 </robot>

Commit message: solved spawning robotiq gripper and controllers

File: urdf/camera.xacro (robot description, xacro)
@@ -1,4 +1,7 @@
 <?xml version="1.0"?>
 <robot xmlns:xacro="http://ros.org/wiki/xacro">
+    <material name="red">
+        <color rgba="1 0 0 1"/>
+    </material>
     <link name="camera_link">
         <inertial>
@@ -18,5 +21,5 @@
         <collision>
             <geometry>
-                <mesh filename="package://ur5_sim/meshes/sensors/camera/kinetic.stl"/>
+                <mesh filename="package://ur5_sim/meshes/sensors/camera/kinetic.dae"/>
             </geometry>
         </collision>
@@ -35,5 +38,13 @@
     </joint>
     <gazebo reference="camera_link">
-        <material>Gazebo/Red</material>
+        <visual>
+            <geometry>
+                <mesh>
+                    <uri>package://ur5_sim/meshes/sensors/camera/kinetic.stl</uri>
+                </mesh>
+            </geometry>
+            <material>Gazebo/Red</material>
+        </visual>
+        <!-- <material>Gazebo/Red</material> -->
         <sensor name="camera" type="depth">
             <pose> 0 0 0 0 0 0 </pose>

File: urdf/robotiq_gripper.ros2_control.xacro (robot description, xacro)
@@ -59,5 +59,5 @@
             </joint>
             <!-- When simulating we need to include the rest of the gripper joints -->
-            <xacro:if value="${use_fake_hardware or sim_isaac or sim_ignition}">
+            <xacro:if value="${sim_gazebo or use_fake_hardware or sim_isaac or sim_ignition}">
                 <joint name="${prefix}robotiq_85_right_knuckle_joint">
                     <param name="mimic">${prefix}robotiq_85_left_knuckle_joint</param>

File: urdf/ur5_camera.urdf.xacro (robot description, xacro)
@@ -1,8 +1,9 @@
 <?xml version="1.0"?>
 <!-- <robot xmlns:xacro="http://wiki.ros.org/xacro" name="$(arg name)"> -->
-<robot xmlns:xacro="http://wiki.ros.org/xacro" name="ur">
+<!-- <robot xmlns:xacro="http://wiki.ros.org/xacro" name="ur"> -->
+<robot xmlns:xacro="http://www.ros.org/wiki/xacro" name="ur">
    <xacro:arg name="name" default="ur"/>
+   <xacro:include filename="$(find ur5_sim)/urdf/camera.xacro"/>
    <xacro:include filename="$(find ur5_sim)/urdf/ur5_macro.xacro"/>
-   <xacro:include filename="$(find ur5_sim)/urdf/camera.xacro"/>
    <!-- possible 'ur_type' values: ur3, ur3e, ur5, ur5e, ur7e, ur10, ur10e, ur12e, ur16e, ur20, ur30 -->
    <!-- the default value should raise an error in case this was called without defining the type -->
